Commit message: Made changes to URDF for proper basic link integration and added static tf between d435_link-->camera_link

File: g1_bringup/urdf/g1_29dof.urdf (robot description, URDF)
Before this commit: robot g1_29dof, 41 links, 40 joints
Links:
- removed link world
- added link base_link
Joints:
- joint floating_base_joint: origin (none) -> xyz=0 0 0.78 rpy=0 0 0; parent world -> base_link

Commit message: Addes the slam and nav launch files in the pkg

File: g1_bringup/urdf/g1_29dof.urdf (robot description, URDF)
Before this commit: robot g1_29dof, 41 links, 40 joints
Joints:
- joint d435_joint: origin xyz=0.0576235 0.01753 0.41987 rpy=0 0.8307767239493009 0 -> xyz=0.0576235 0.01753 0.05 rpy=0 0 0
